Commit message: Restore MoveIt execution with RG2 geometry attached

File: ros2_ws/install/robot_description/share/robot_description/urdf/ur5e_ros.urdf (robot description, URDF)
Before this commit: robot ur5e, 9 links, 8 joints
Links:
- added link onrobot_rg2_base_link, mass 0.09; collision mesh filename=package://robot_description/meshes/onrobot_rg2ft/collision/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 scale=0.001 0.001 0.001; visual mesh filename=package://robot_description/meshes/onrobot_rg2ft/visual/ang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 scale=0.001 0.001 0.001
- added link onrobot_rg2_body_link, mass 0.65; collision mesh filename=package://onrobot_description/meshes/rg2_v1/collision/body.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; visual mesh filename=package://onrobot_description/meshes/rg2_v1/visual/body.stl
- added link onrobot_rg2_finger_1_finger_tip_link, mass 0.001; collision mesh filename=package://onrobot_description/meshes/rg2_v1/collision/finge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; visual mesh filename=package://onrobot_description/meshes/rg2_v1/visual/finger_t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
- added link onrobot_rg2_finger_1_flex_finger_link, mass 0.001; collision mesh filename=package://onrobot_description/meshes/rg2_v1/collision/flex_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; visual mesh filename=package://onrobot_description/meshes/rg2_v1/visual/flex_fin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
- added link onrobot_rg2_finger_1_moment_arm_link, mass 0.001; collision mesh filename=package://onrobot_description/meshes/rg2_v1/collision/momen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; visual mesh filename=package://onrobot_description/meshes/rg2_v1/visual/moment_a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
- added link onrobot_rg2_finger_1_origin, mass 0.001
- added link onrobot_rg2_finger_1_truss_arm_link, mass 0.001; collision mesh filename=package://onrobot_description/meshes/rg2_v1/collision/truss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; visual mesh filename=package://onrobot_description/meshes/rg2_v1/visual/truss_ar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
- added link onrobot_rg2_finger_2_finger_tip_link, mass 0.001; collision mesh filename=package://onrobot_description/meshes/rg2_v1/collision/finge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; visual mesh filename=package://onrobot_description/meshes/rg2_v1/visual/finger_t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
- added link onrobot_rg2_finger_2_flex_finger_link, mass 0.001; collision mesh filename=package://onrobot_description/meshes/rg2_v1/collision/flex_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; visual mesh filename=package://onrobot_description/meshes/rg2_v1/visual/flex_fin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
- added link onrobot_rg2_finger_2_moment_arm_link, mass 0.001; collision mesh filename=package://onrobot_description/meshes/rg2_v1/collision/momen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; visual mesh filename=package://onrobot_description/meshes/rg2_v1/visual/moment_a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
- added link onrobot_rg2_finger_2_origin, mass 0.001
- added link onrobot_rg2_finger_2_truss_arm_link, mass 0.001; collision mesh filename=package://onrobot_description/meshes/rg2_v1/collision/truss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; visual mesh filename=package://onrobot_description/meshes/rg2_v1/visual/truss_ar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
- added link onrobot_rg2_grasp_frame, mass 1e-6
Joints:
- added joint Gripper_joint: type fixed, parent wrist_3_link, child onrobot_rg2_base_link, origin xyz=0 0 0 rpy=0 0 0
- added joint onrobot_rg2_base_to_body_joint: type fixed, parent onrobot_rg2_base_link, child onrobot_rg2_body_link, origin xyz=0 0 0.05 rpy=0 0 0
- added joint onrobot_rg2_body_to_finger_1_origin_joint: type fixed, parent onrobot_rg2_body_link, child onrobot_rg2_finger_1_origin, origin xyz=0 0 0 rpy=0 0 0
- added joint onrobot_rg2_body_to_finger_2_origin_joint: type fixed, parent onrobot_rg2_body_link, child onrobot_rg2_finger_2_origin, origin xyz=0 0 0 rpy=0 0 3.141592653589793
- added joint onrobot_rg2_body_to_grasp_frame_joint: type fixed, parent onrobot_rg2_body_link, child onrobot_rg2_grasp_frame, origin xyz=0 0 0.14 rpy=0 0 0
- added joint onrobot_rg2_finger_1_finger_tip_to_flex_finger_joint: type fixed, parent onrobot_rg2_finger_1_finger_tip_link, child onrobot_rg2_finger_1_flex_finger_link, origin xyz=0.03059 0 0.0172 rpy=0 0 0
- added joint onrobot_rg2_finger_1_origin_to_moment_arm_joint: type fixed, parent onrobot_rg2_finger_1_origin, child onrobot_rg2_finger_1_moment_arm_link, origin xyz=-0.017 0 0.055 rpy=0 -0.772 0
- added joint onrobot_rg2_finger_1_origin_to_truss_arm_joint: type fixed, parent onrobot_rg2_finger_1_origin, child onrobot_rg2_finger_1_truss_arm_link, origin xyz=-0.0075 0 0.0715 rpy=0 -0.772 0
- added joint onrobot_rg2_finger_1_truss_arm_to_finger_tip_joint: type fixed, parent onrobot_rg2_finger_1_truss_arm_link, child onrobot_rg2_finger_1_finger_tip_link, origin xyz=-0.0256 0 0.04868 rpy=0 0.772 0
- added joint onrobot_rg2_finger_2_finger_tip_to_flex_finger_joint: type fixed, parent onrobot_rg2_finger_2_finger_tip_link, child onrobot_rg2_finger_2_flex_finger_link, origin xyz=0.03059 0 0.0172 rpy=0 0 0
- added joint onrobot_rg2_finger_2_origin_to_moment_arm_joint: type fixed, parent onrobot_rg2_finger_2_origin, child onrobot_rg2_finger_2_moment_arm_link, origin xyz=-0.017 0 0.055 rpy=0 -0.772 0
- added joint onrobot_rg2_finger_2_origin_to_truss_arm_joint: type fixed, parent onrobot_rg2_finger_2_origin, child onrobot_rg2_finger_2_truss_arm_link, origin xyz=-0.0075 0 0.0715 rpy=0 -0.772 0
- added joint onrobot_rg2_finger_2_truss_arm_to_finger_tip_joint: type fixed, parent onrobot_rg2_finger_2_truss_arm_link, child onrobot_rg2_finger_2_finger_tip_link, origin xyz=-0.0256 0 0.04868 rpy=0 0.772 0

File: ros2_ws/src/robot_description/urdf/ur5e_ros.urdf (robot description, URDF)
Before this commit: robot ur5e, 22 links, 22 joints
Joints:
- removed joint onrobot_rg2_base_to_bracket_joint
- removed joint onrobot_rg2_bracket_to_body_joint
- added joint onrobot_rg2_base_to_body_joint: type fixed, parent onrobot_rg2_base_link, child onrobot_rg2_body_link, origin xyz=0 0 0.05 rpy=0 0 0
