Commit message: Refactor RG2 gripper bridge to enhance joint control by changing joint types to revolute, adding limits, dynamics, and mimic settings. Update configuration files and launch scripts to support new gripper command topics and presets, improving usability and integration with the simulation environment. Add a script for inspecting URDF joints to ensure correct configurations.

File: generated_urdf/rg2_only/rg2_only.urdf (robot description, URDF)
Before this commit: robot onrobot_rg2, 13 links, 12 joints
Joints:
- joint onrobot_rg2_body_to_finger_1_origin_joint: axis (none) -> -0.0 0.999949 -0.010122; limit (none) -> lower=0.0 upper=1.18 effort=50.0 velocity=2.0; type fixed -> revolute
- joint onrobot_rg2_body_to_finger_2_origin_joint: axis (none) -> -0.0 0.999949 -0.010122; limit (none) -> lower=-1.19 upper=1.19 effort=50.0 velocity=2.0; mimic (none) -> joint=onrobot_rg2_body_to_finger_1_origin_joint multiplier=1 offset=0; type fixed -> revolute
- joint onrobot_rg2_finger_1_origin_to_moment_arm_joint: axis (none) -> -0.0 0.999949 -0.010122; limit (none) -> lower=-1.19 upper=1.19 effort=50.0 velocity=2.0; mimic (none) -> joint=onrobot_rg2_body_to_finger_1_origin_joint multiplier=-1 offset=0; type fixed -> revolute
- joint onrobot_rg2_finger_1_origin_to_truss_arm_joint: axis (none) -> -0.0 0.999949 -0.010122; limit (none) -> lower=-1.19 upper=1.19 effort=50.0 velocity=2.0; mimic (none) -> joint=onrobot_rg2_body_to_finger_1_origin_joint multiplier=-1 offset=0; type fixed -> revolute
- joint onrobot_rg2_finger_1_truss_arm_to_finger_tip_joint: axis (none) -> 0.0 -0.999949 0.010122; limit (none) -> lower=-1.19 upper=1.19 effort=50.0 velocity=2.0; mimic (none) -> joint=onrobot_rg2_body_to_finger_1_origin_joint multiplier=-1 offset=0; type fixed -> revolute
- joint onrobot_rg2_finger_2_origin_to_moment_arm_joint: axis (none) -> -0.0 0.999949 -0.010122; limit (none) -> lower=-1.19 upper=1.19 effort=50.0 velocity=2.0; mimic (none) -> joint=onrobot_rg2_body_to_finger_1_origin_joint multiplier=-1 offset=0; type fixed -> revolute
- joint onrobot_rg2_finger_2_origin_to_truss_arm_joint: axis (none) -> -0.0 0.999949 -0.010122; limit (none) -> lower=-1.19 upper=1.19 effort=50.0 velocity=2.0; mimic (none) -> joint=onrobot_rg2_body_to_finger_1_origin_joint multiplier=-1 offset=0; type fixed -> revolute
- joint onrobot_rg2_finger_2_truss_arm_to_finger_tip_joint: axis (none) -> 0.0 0.999949 -0.010122; limit (none) -> lower=-1.19 upper=1.19 effort=50.0 velocity=2.0; mimic (none) -> joint=onrobot_rg2_body_to_finger_1_origin_joint multiplier=-1 offset=0; type fixed -> revolute

File: generated_urdf/rg2_only/rg2_only_isaac.urdf (robot description, URDF)
Before this commit: robot onrobot_rg2, 13 links, 12 joints
Joints:
- joint onrobot_rg2_finger_1_origin_to_moment_arm_joint: limit lower=-1.19 upper=0.01 effort=50.0 velocity=2.0 -> lower=-1.19 upper=1.19 effort=50.0 velocity=2.0; mimic joint=onrobot_rg2_body_to_finger_1_origin_joint multiplier=-1 offset=0 -> joint=onrobot_rg2_body_to_finger_1_origin_joint multiplier=-1.0 offset=0
- joint onrobot_rg2_finger_1_origin_to_truss_arm_joint: limit lower=-1.19 upper=0.01 effort=50.0 velocity=2.0 -> lower=-1.19 upper=1.19 effort=50.0 velocity=2.0; mimic joint=onrobot_rg2_body_to_finger_1_origin_joint multiplier=-1 offset=0 -> joint=onrobot_rg2_body_to_finger_1_origin_joint multiplier=-1.0 offset=0
- joint onrobot_rg2_finger_1_truss_arm_to_finger_tip_joint: limit lower=-1.19 upper=0.01 effort=50.0 velocity=2.0 -> lower=-1.19 upper=1.19 effort=50.0 velocity=2.0; mimic joint=onrobot_rg2_body_to_finger_1_origin_joint multiplier=-1 offset=0 -> joint=onrobot_rg2_body_to_finger_1_origin_joint multiplier=-1.0 offset=0
- joint onrobot_rg2_finger_2_origin_to_moment_arm_joint: limit lower=-1.19 upper=0.01 effort=50.0 velocity=2.0 -> lower=-1.19 upper=1.19 effort=50.0 velocity=2.0; mimic joint=onrobot_rg2_body_to_finger_1_origin_joint multiplier=-1 offset=0 -> joint=onrobot_rg2_body_to_finger_1_origin_joint multiplier=-1.0 offset=0
- joint onrobot_rg2_finger_2_origin_to_truss_arm_joint: limit lower=-1.19 upper=0.01 effort=50.0 velocity=2.0 -> lower=-1.19 upper=1.19 effort=50.0 velocity=2.0; mimic joint=onrobot_rg2_body_to_finger_1_origin_joint multiplier=-1 offset=0 -> joint=onrobot_rg2_body_to_finger_1_origin_joint multiplier=-1.0 offset=0
- joint onrobot_rg2_finger_2_truss_arm_to_finger_tip_joint: limit lower=-1.19 upper=0.01 effort=50.0 velocity=2.0 -> lower=-1.19 upper=1.19 effort=50.0 velocity=2.0; mimic joint=onrobot_rg2_body_to_finger_1_origin_joint multiplier=-1 offset=0 -> joint=onrobot_rg2_body_to_finger_1_origin_joint multiplier=-1.0 offset=0

File: ros2_ws/src/robot_description/urdf/ur5e_ros.urdf (robot description, URDF)
Before this commit: robot ur5e, 22 links, 21 joints
Joints:
- joint onrobot_rg2_body_to_finger_1_origin_joint: axis (none) -> -0.0 0.999949 -0.010122; limit (none) -> lower=0.0 upper=1.18 effort=50.0 velocity=2.0; type fixed -> revolute
- joint onrobot_rg2_body_to_finger_2_origin_joint: axis (none) -> -0.0 0.999949 -0.010122; limit (none) -> lower=-1.19 upper=1.19 effort=50.0 velocity=2.0; mimic (none) -> joint=onrobot_rg2_body_to_finger_1_origin_joint multiplier=1 offset=0; type fixed -> revolute
- joint onrobot_rg2_finger_1_origin_to_moment_arm_joint: axis (none) -> -0.0 0.999949 -0.010122; limit (none) -> lower=-1.19 upper=1.19 effort=50.0 velocity=2.0; mimic (none) -> joint=onrobot_rg2_body_to_finger_1_origin_joint multiplier=-1 offset=0; type fixed -> revolute
- joint onrobot_rg2_finger_1_origin_to_truss_arm_joint: axis (none) -> -0.0 0.999949 -0.010122; limit (none) -> lower=-1.19 upper=1.19 effort=50.0 velocity=2.0; mimic (none) -> joint=onrobot_rg2_body_to_finger_1_origin_joint multiplier=-1 offset=0; type fixed -> revolute
- joint onrobot_rg2_finger_1_truss_arm_to_finger_tip_joint: axis (none) -> 0.0 -0.999949 0.010122; limit (none) -> lower=-1.19 upper=1.19 effort=50.0 velocity=2.0; mimic (none) -> joint=onrobot_rg2_body_to_finger_1_origin_joint multiplier=-1 offset=0; type fixed -> revolute
- joint onrobot_rg2_finger_2_origin_to_moment_arm_joint: axis (none) -> -0.0 0.999949 -0.010122; limit (none) -> lower=-1.19 upper=1.19 effort=50.0 velocity=2.0; mimic (none) -> joint=onrobot_rg2_body_to_finger_1_origin_joint multiplier=-1 offset=0; type fixed -> revolute
- joint onrobot_rg2_finger_2_origin_to_truss_arm_joint: axis (none) -> -0.0 0.999949 -0.010122; limit (none) -> lower=-1.19 upper=1.19 effort=50.0 velocity=2.0; mimic (none) -> joint=onrobot_rg2_body_to_finger_1_origin_joint multiplier=-1 offset=0; type fixed -> revolute
- joint onrobot_rg2_finger_2_truss_arm_to_finger_tip_joint: axis (none) -> 0.0 0.999949 -0.010122; limit (none) -> lower=-1.19 upper=1.19 effort=50.0 velocity=2.0; mimic (none) -> joint=onrobot_rg2_body_to_finger_1_origin_joint multiplier=-1 offset=0; type fixed -> revolute

Commit message: RG2 Gripper Dynamics and Kinematics finalized in URDF.

File: generated_urdf/rg2_only/rg2_only.urdf (robot description, URDF)
Before this commit: robot onrobot_rg2, 13 links, 12 joints
Joints:
- joint onrobot_rg2_base_to_body_joint: origin xyz=0 0 0.05 rpy=0 0 0 -> xyz=0.0 0.0 0.05 rpy=0.0 0.0 0.0
- joint onrobot_rg2_body_to_finger_1_origin_joint: axis -0.0 0.999949 -0.010122 -> (none); limit lower=0.0 upper=1.18 effort=50.0 velocity=2.0 -> (none); type revolute -> fixed
- joint onrobot_rg2_body_to_finger_2_origin_joint: axis -0.0 0.999949 -0.010122 -> (none); limit lower=-1.19 upper=1.19 effort=50.0 velocity=2.0 -> (none); mimic joint=onrobot_rg2_body_to_finger_1_origin_joint multiplier=1 offset=0 -> (none); type revolute -> fixed
- joint onrobot_rg2_body_to_grasp_frame_joint: origin xyz=0 0 0.14 rpy=0 0 0 -> xyz=0.0 0.0 0.14 rpy=0.0 0.0 0.0
- joint onrobot_rg2_finger_1_finger_tip_to_flex_finger_joint: origin xyz=0.03059 0 0.0172 rpy=0 0 0 -> xyz=0.03059 0.0 0.0172 rpy=0.0 0.0 0.0
- joint onrobot_rg2_finger_1_origin_to_moment_arm_joint: axis -0.0 0.999949 -0.010122 -> 0 1 0; limit lower=-1.19 upper=1.19 effort=50.0 velocity=2.0 -> lower=0.0 upper=1.3 effort=10.0 velocity=50.0; mimic joint=onrobot_rg2_body_to_finger_1_origin_joint multiplier=-1 offset=0 -> (none); origin xyz=-0.017 0 0.055 rpy=0 -0.772 0 -> xyz=-0.017 0.0 0.055 rpy=0.0 -0.772 0.0
- joint onrobot_rg2_finger_1_origin_to_truss_arm_joint: axis -0.0 0.999949 -0.010122 -> 0 1 0; limit lower=-1.19 upper=1.19 effort=50.0 velocity=2.0 -> lower=0.0 upper=1.3 effort=10.0 velocity=50.0; mimic joint=onrobot_rg2_body_to_finger_1_origin_joint multiplier=-1 offset=0 -> joint=onrobot_rg2_finger_1_origin_to_moment_arm_joint multiplier=1 offset=0; origin xyz=-0.0075 0 0.0715 rpy=0 -0.772 0 -> xyz=-0.0075 0.0 0.0715 rpy=0.0 -0.772 0.0
- joint onrobot_rg2_finger_1_truss_arm_to_finger_tip_joint: axis 0.0 -0.999949 0.010122 -> 0 -1 0; limit lower=-1.19 upper=1.19 effort=50.0 velocity=2.0 -> lower=0.0 upper=1.3 effort=10.0 velocity=50.0; mimic joint=onrobot_rg2_body_to_finger_1_origin_joint multiplier=-1 offset=0 -> joint=onrobot_rg2_finger_1_origin_to_moment_arm_joint multiplier=1 offset=0; origin xyz=-0.0256 0 0.04868 rpy=0 0.772 0 -> xyz=-0.0256 0.0 0.04868 rpy=0.0 0.772 0.0
- joint onrobot_rg2_finger_2_finger_tip_to_flex_finger_joint: origin xyz=0.03059 0 0.0172 rpy=0 0 0 -> xyz=0.03059 0.0 0.0172 rpy=0.0 0.0 0.0
- joint onrobot_rg2_finger_2_origin_to_moment_arm_joint: axis -0.0 0.999949 -0.010122 -> 0 1 0; limit lower=-1.19 upper=1.19 effort=50.0 velocity=2.0 -> lower=0.0 upper=1.3 effort=10.0 velocity=50.0; mimic joint=onrobot_rg2_body_to_finger_1_origin_joint multiplier=-1 offset=0 -> joint=onrobot_rg2_finger_1_origin_to_moment_arm_joint multiplier=1 offset=0; origin xyz=-0.017 0 0.055 rpy=0 -0.772 0 -> xyz=-0.017 0.0 0.055 rpy=0.0 -0.772 0.0
- joint onrobot_rg2_finger_2_origin_to_truss_arm_joint: axis -0.0 0.999949 -0.010122 -> 0 1 0; limit lower=-1.19 upper=1.19 effort=50.0 velocity=2.0 -> lower=0.0 upper=1.3 effort=10.0 velocity=50.0; mimic joint=onrobot_rg2_body_to_finger_1_origin_joint multiplier=-1 offset=0 -> joint=onrobot_rg2_finger_1_origin_to_moment_arm_joint multiplier=1 offset=0; origin xyz=-0.0075 0 0.0715 rpy=0 -0.772 0 -> xyz=-0.0075 0.0 0.0715 rpy=0.0 -0.772 0.0
- joint onrobot_rg2_finger_2_truss_arm_to_finger_tip_joint: axis 0.0 0.999949 -0.010122 -> 0 -1 0; limit lower=-1.19 upper=1.19 effort=50.0 velocity=2.0 -> lower=0.0 upper=1.3 effort=10.0 velocity=50.0; mimic joint=onrobot_rg2_body_to_finger_1_origin_joint multiplier=-1 offset=0 -> joint=onrobot_rg2_finger_1_origin_to_moment_arm_joint multiplier=1 offset=0; origin xyz=-0.0256 0 0.04868 rpy=0 0.772 0 -> xyz=-0.0256 0.0 0.04868 rpy=0.0 0.772 0.0

File: generated_urdf/rg2_only/rg2_only_isaac.urdf (robot description, URDF)
Before this commit: robot onrobot_rg2, 13 links, 12 joints
Joints:
- joint onrobot_rg2_base_to_body_joint: origin xyz=0 0 0.05 rpy=0 0 0 -> xyz=0.0 0.0 0.05 rpy=0.0 0.0 0.0
- joint onrobot_rg2_body_to_finger_1_origin_joint: axis -0.0 0.999949 -0.010122 -> (none); limit lower=0.0 upper=1.18 effort=50.0 velocity=2.0 -> (none); type revolute -> fixed
- joint onrobot_rg2_body_to_finger_2_origin_joint: axis -0.0 0.999949 -0.010122 -> (none); limit lower=-1.19 upper=1.19 effort=50.0 velocity=2.0 -> (none); mimic joint=onrobot_rg2_body_to_finger_1_origin_joint multiplier=1.0 offset=0 -> (none); type revolute -> fixed
- joint onrobot_rg2_body_to_grasp_frame_joint: origin xyz=0 0 0.14 rpy=0 0 0 -> xyz=0.0 0.0 0.14 rpy=0.0 0.0 0.0
- joint onrobot_rg2_finger_1_finger_tip_to_flex_finger_joint: origin xyz=0.03059 0 0.0172 rpy=0 0 0 -> xyz=0.03059 0.0 0.0172 rpy=0.0 0.0 0.0
- joint onrobot_rg2_finger_1_origin_to_moment_arm_joint: axis -0.0 0.999949 -0.010122 -> 0 1 0; limit lower=-1.19 upper=1.19 effort=50.0 velocity=2.0 -> lower=0.0 upper=1.3 effort=10.0 velocity=50.0; mimic joint=onrobot_rg2_body_to_finger_1_origin_joint multiplier=-1.0 offset=0 -> (none); origin xyz=-0.017 0 0.055 rpy=0 -0.772 0 -> xyz=-0.017 0.0 0.055 rpy=0.0 -0.772 0.0
- joint onrobot_rg2_finger_1_origin_to_truss_arm_joint: axis -0.0 0.999949 -0.010122 -> 0 1 0; limit lower=-1.19 upper=1.19 effort=50.0 velocity=2.0 -> lower=0.0 upper=1.3 effort=10.0 velocity=50.0; mimic joint=onrobot_rg2_body_to_finger_1_origin_joint multiplier=-1.0 offset=0 -> joint=onrobot_rg2_finger_1_origin_to_moment_arm_joint multiplier=1 offset=0; origin xyz=-0.0075 0 0.0715 rpy=0 -0.772 0 -> xyz=-0.0075 0.0 0.0715 rpy=0.0 -0.772 0.0
- joint onrobot_rg2_finger_1_truss_arm_to_finger_tip_joint: axis 0.0 -0.999949 0.010122 -> 0 -1 0; limit lower=-1.19 upper=1.19 effort=50.0 velocity=2.0 -> lower=0.0 upper=1.3 effort=10.0 velocity=50.0; mimic joint=onrobot_rg2_body_to_finger_1_origin_joint multiplier=-1.0 offset=0 -> joint=onrobot_rg2_finger_1_origin_to_moment_arm_joint multiplier=1 offset=0; origin xyz=-0.0256 0 0.04868 rpy=0 0.772 0 -> xyz=-0.0256 0.0 0.04868 rpy=0.0 0.772 0.0
- joint onrobot_rg2_finger_2_finger_tip_to_flex_finger_joint: origin xyz=0.03059 0 0.0172 rpy=0 0 0 -> xyz=0.03059 0.0 0.0172 rpy=0.0 0.0 0.0
- joint onrobot_rg2_finger_2_origin_to_moment_arm_joint: axis -0.0 0.999949 -0.010122 -> 0 1 0; limit lower=-1.19 upper=1.19 effort=50.0 velocity=2.0 -> lower=0.0 upper=1.3 effort=10.0 velocity=50.0; mimic joint=onrobot_rg2_body_to_finger_1_origin_joint multiplier=-1.0 offset=0 -> joint=onrobot_rg2_finger_1_origin_to_moment_arm_joint multiplier=1 offset=0; origin xyz=-0.017 0 0.055 rpy=0 -0.772 0 -> xyz=-0.017 0.0 0.055 rpy=0.0 -0.772 0.0
- joint onrobot_rg2_finger_2_origin_to_truss_arm_joint: axis -0.0 0.999949 -0.010122 -> 0 1 0; limit lower=-1.19 upper=1.19 effort=50.0 velocity=2.0 -> lower=0.0 upper=1.3 effort=10.0 velocity=50.0; mimic joint=onrobot_rg2_body_to_finger_1_origin_joint multiplier=-1.0 offset=0 -> joint=onrobot_rg2_finger_1_origin_to_moment_arm_joint multiplier=1 offset=0; origin xyz=-0.0075 0 0.0715 rpy=0 -0.772 0 -> xyz=-0.0075 0.0 0.0715 rpy=0.0 -0.772 0.0
- joint onrobot_rg2_finger_2_truss_arm_to_finger_tip_joint: axis 0.0 0.999949 -0.010122 -> 0 -1 0; limit lower=-1.19 upper=1.19 effort=50.0 velocity=2.0 -> lower=0.0 upper=1.3 effort=10.0 velocity=50.0; mimic joint=onrobot_rg2_body_to_finger_1_origin_joint multiplier=-1.0 offset=0 -> joint=onrobot_rg2_finger_1_origin_to_moment_arm_joint multiplier=1 offset=0; origin xyz=-0.0256 0 0.04868 rpy=0 0.772 0 -> xyz=-0.0256 0.0 0.04868 rpy=0.0 0.772 0.0

File: ros2_ws/src/robot_description/urdf/ur5e_ros.urdf (robot description, URDF)
Before this commit: robot ur5e, 22 links, 21 joints
Joints:
- joint onrobot_rg2_base_to_body_joint: origin xyz=0 0 0.05 rpy=0 0 0 -> xyz=0.0 0.0 0.05 rpy=0.0 0.0 0.0
- joint onrobot_rg2_body_to_finger_1_origin_joint: axis -0.0 0.999949 -0.010122 -> (none); limit lower=0.0 upper=1.18 effort=50.0 velocity=2.0 -> (none); type revolute -> fixed
- joint onrobot_rg2_body_to_finger_2_origin_joint: axis -0.0 0.999949 -0.010122 -> (none); limit lower=-1.19 upper=1.19 effort=50.0 velocity=2.0 -> (none); mimic joint=onrobot_rg2_body_to_finger_1_origin_joint multiplier=1 offset=0 -> (none); type revolute -> fixed
- joint onrobot_rg2_body_to_grasp_frame_joint: origin xyz=0 0 0.14 rpy=0 0 0 -> xyz=0.0 0.0 0.14 rpy=0.0 0.0 0.0
- joint onrobot_rg2_finger_1_finger_tip_to_flex_finger_joint: origin xyz=0.03059 0 0.0172 rpy=0 0 0 -> xyz=0.03059 0.0 0.0172 rpy=0.0 0.0 0.0
- joint onrobot_rg2_finger_1_origin_to_moment_arm_joint: axis -0.0 0.999949 -0.010122 -> 0 1 0; limit lower=-1.19 upper=1.19 effort=50.0 velocity=2.0 -> lower=0.0 upper=1.3 effort=10.0 velocity=50.0; mimic joint=onrobot_rg2_body_to_finger_1_origin_joint multiplier=-1 offset=0 -> (none); origin xyz=-0.017 0 0.055 rpy=0 -0.772 0 -> xyz=-0.017 0.0 0.055 rpy=0.0 -0.772 0.0
- joint onrobot_rg2_finger_1_origin_to_truss_arm_joint: axis -0.0 0.999949 -0.010122 -> 0 1 0; limit lower=-1.19 upper=1.19 effort=50.0 velocity=2.0 -> lower=0.0 upper=1.3 effort=10.0 velocity=50.0; mimic joint=onrobot_rg2_body_to_finger_1_origin_joint multiplier=-1 offset=0 -> joint=onrobot_rg2_finger_1_origin_to_moment_arm_joint multiplier=1 offset=0; origin xyz=-0.0075 0 0.0715 rpy=0 -0.772 0 -> xyz=-0.0075 0.0 0.0715 rpy=0.0 -0.772 0.0
- joint onrobot_rg2_finger_1_truss_arm_to_finger_tip_joint: axis 0.0 -0.999949 0.010122 -> 0 -1 0; limit lower=-1.19 upper=1.19 effort=50.0 velocity=2.0 -> lower=0.0 upper=1.3 effort=10.0 velocity=50.0; mimic joint=onrobot_rg2_body_to_finger_1_origin_joint multiplier=-1 offset=0 -> joint=onrobot_rg2_finger_1_origin_to_moment_arm_joint multiplier=1 offset=0; origin xyz=-0.0256 0 0.04868 rpy=0 0.772 0 -> xyz=-0.0256 0.0 0.04868 rpy=0.0 0.772 0.0
- joint onrobot_rg2_finger_2_finger_tip_to_flex_finger_joint: origin xyz=0.03059 0 0.0172 rpy=0 0 0 -> xyz=0.03059 0.0 0.0172 rpy=0.0 0.0 0.0
- joint onrobot_rg2_finger_2_origin_to_moment_arm_joint: axis -0.0 0.999949 -0.010122 -> 0 1 0; limit lower=-1.19 upper=1.19 effort=50.0 velocity=2.0 -> lower=0.0 upper=1.3 effort=10.0 velocity=50.0; mimic joint=onrobot_rg2_body_to_finger_1_origin_joint multiplier=-1 offset=0 -> joint=onrobot_rg2_finger_1_origin_to_moment_arm_joint multiplier=1 offset=0; origin xyz=-0.017 0 0.055 rpy=0 -0.772 0 -> xyz=-0.017 0.0 0.055 rpy=0.0 -0.772 0.0
- joint onrobot_rg2_finger_2_origin_to_truss_arm_joint: axis -0.0 0.999949 -0.010122 -> 0 1 0; limit lower=-1.19 upper=1.19 effort=50.0 velocity=2.0 -> lower=0.0 upper=1.3 effort=10.0 velocity=50.0; mimic joint=onrobot_rg2_body_to_finger_1_origin_joint multiplier=-1 offset=0 -> joint=onrobot_rg2_finger_1_origin_to_moment_arm_joint multiplier=1 offset=0; origin xyz=-0.0075 0 0.0715 rpy=0 -0.772 0 -> xyz=-0.0075 0.0 0.0715 rpy=0.0 -0.772 0.0
- joint onrobot_rg2_finger_2_truss_arm_to_finger_tip_joint: axis 0.0 0.999949 -0.010122 -> 0 -1 0; limit lower=-1.19 upper=1.19 effort=50.0 velocity=2.0 -> lower=0.0 upper=1.3 effort=10.0 velocity=50.0; mimic joint=onrobot_rg2_body_to_finger_1_origin_joint multiplier=-1 offset=0 -> joint=onrobot_rg2_finger_1_origin_to_moment_arm_joint multiplier=1 offset=0; origin xyz=-0.0256 0 0.04868 rpy=0 0.772 0 -> xyz=-0.0256 0.0 0.04868 rpy=0.0 0.772 0.0
