Commit message: Refactor RG2 gripper joints in URDF to use revolute type, adding limits, dynamics, and mimic settings for improved control. Update CMakeLists.txt to install RG2 gripper bridge script and enhance README.md with detailed usage instructions for the RG2 gripper bridge, including command topics and configuration options.

File: generated_urdf/rg2_only/rg2_only_isaac.urdf (robot description, URDF)
Before this commit: robot onrobot_rg2, 13 links, 12 joints
Joints:
- joint onrobot_rg2_body_to_finger_1_origin_joint: axis (none) -> -0.0 0.999949 -0.010122; limit (none) -> lower=0.0 upper=1.18 effort=50.0 velocity=2.0; type fixed -> revolute
- joint onrobot_rg2_body_to_finger_2_origin_joint: axis (none) -> -0.0 0.999949 -0.010122; limit (none) -> lower=-1.19 upper=1.19 effort=50.0 velocity=2.0; mimic (none) -> joint=onrobot_rg2_body_to_finger_1_origin_joint multiplier=1.0 offset=0; type fixed -> revolute
- joint onrobot_rg2_finger_1_origin_to_moment_arm_joint: axis (none) -> -0.0 0.999949 -0.010122; limit (none) -> lower=-1.19 upper=0.01 effort=50.0 velocity=2.0; mimic (none) -> joint=onrobot_rg2_body_to_finger_1_origin_joint multiplier=-1 offset=0; type fixed -> revolute
- joint onrobot_rg2_finger_1_origin_to_truss_arm_joint: axis (none) -> -0.0 0.999949 -0.010122; limit (none) -> lower=-1.19 upper=0.01 effort=50.0 velocity=2.0; mimic (none) -> joint=onrobot_rg2_body_to_finger_1_origin_joint multiplier=-1 offset=0; type fixed -> revolute
- joint onrobot_rg2_finger_1_truss_arm_to_finger_tip_joint: axis (none) -> 0.0 -0.999949 0.010122; limit (none) -> lower=-1.19 upper=0.01 effort=50.0 velocity=2.0; mimic (none) -> joint=onrobot_rg2_body_to_finger_1_origin_joint multiplier=-1 offset=0; type fixed -> revolute
- joint onrobot_rg2_finger_2_origin_to_moment_arm_joint: axis (none) -> -0.0 0.999949 -0.010122; limit (none) -> lower=-1.19 upper=0.01 effort=50.0 velocity=2.0; mimic (none) -> joint=onrobot_rg2_body_to_finger_1_origin_joint multiplier=-1 offset=0; type fixed -> revolute
- joint onrobot_rg2_finger_2_origin_to_truss_arm_joint: axis (none) -> -0.0 0.999949 -0.010122; limit (none) -> lower=-1.19 upper=0.01 effort=50.0 velocity=2.0; mimic (none) -> joint=onrobot_rg2_body_to_finger_1_origin_joint multiplier=-1 offset=0; type fixed -> revolute
- joint onrobot_rg2_finger_2_truss_arm_to_finger_tip_joint: axis (none) -> 0.0 0.999949 -0.010122; limit (none) -> lower=-1.19 upper=0.01 effort=50.0 velocity=2.0; mimic (none) -> joint=onrobot_rg2_body_to_finger_1_origin_joint multiplier=-1 offset=0; type fixed -> revolute

Commit message: Add RG2 Good USD file, update RG2 MN USD file, and remove RG2 test USD file. Adjust joint limits in URDF for RG2 gripper to improve control precision.

File: generated_urdf/rg2_only/rg2_only_isaac.urdf (robot description, URDF)
Before this commit: robot onrobot_rg2, 13 links, 12 joints
Joints:
- joint onrobot_rg2_finger_1_origin_to_moment_arm_joint: limit lower=0.0 upper=1.3 effort=10.0 velocity=50.0 -> lower=0.0 upper=1.218 effort=10.0 velocity=50.0
- joint onrobot_rg2_finger_1_origin_to_truss_arm_joint: limit lower=0.0 upper=1.3 effort=10.0 velocity=50.0 -> lower=0.0 upper=1.218 effort=10.0 velocity=50.0
- joint onrobot_rg2_finger_1_truss_arm_to_finger_tip_joint: limit lower=0.0 upper=1.3 effort=10.0 velocity=50.0 -> lower=0.0 upper=1.218 effort=10.0 velocity=50.0
- joint onrobot_rg2_finger_2_origin_to_moment_arm_joint: limit lower=0.0 upper=1.3 effort=10.0 velocity=50.0 -> lower=0.0 upper=1.218 effort=10.0 velocity=50.0
- joint onrobot_rg2_finger_2_origin_to_truss_arm_joint: limit lower=0.0 upper=1.3 effort=10.0 velocity=50.0 -> lower=0.0 upper=1.218 effort=10.0 velocity=50.0
- joint onrobot_rg2_finger_2_truss_arm_to_finger_tip_joint: limit lower=0.0 upper=1.3 effort=10.0 velocity=50.0 -> lower=0.0 upper=1.218 effort=10.0 velocity=50.0

Commit message: Add OnRobot RG2 model description package with URDF and mesh files for simulation. Include CMake and package configuration, along with RViz visualization settings for improved usability. Update joint definitions and parameters for accurate representation in simulation environments.

File: generated_urdf/rg2_only/rg2_only_isaac.urdf (robot description, URDF)
Before this commit: robot onrobot_rg2, 13 links, 12 joints
Links:
- removed link onrobot_rg2_base_link
- removed link onrobot_rg2_body_link
- removed link onrobot_rg2_finger_1_finger_tip_link
- removed link onrobot_rg2_finger_1_flex_finger_link
- removed link onrobot_rg2_finger_1_moment_arm_link
- removed link onrobot_rg2_finger_1_origin
- removed link onrobot_rg2_finger_1_truss_arm_link
- removed link onrobot_rg2_finger_2_finger_tip_link
- removed link onrobot_rg2_finger_2_flex_finger_link
- removed link onrobot_rg2_finger_2_moment_arm_link
- removed link onrobot_rg2_finger_2_origin
- removed link onrobot_rg2_finger_2_truss_arm_link
- removed link onrobot_rg2_grasp_frame
- added link base_link, mass 0.7; collision mesh filename=file:///home/mohammadnsr1/watchdog/WatchDog_V1/ros2_ws/src/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; visual mesh filename=file:///home/mohammadnsr1/watchdog/WatchDog_V1/ros2_ws/src/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
- added link left_inner_finger, mass 0.05; collision mesh filename=file:///home/mohammadnsr1/watchdog/WatchDog_V1/ros2_ws/src/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; visual mesh filename=file:///home/mohammadnsr1/watchdog/WatchDog_V1/ros2_ws/src/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
- added link left_inner_knuckle, mass 0.05; collision mesh filename=file:///home/mohammadnsr1/watchdog/WatchDog_V1/ros2_ws/src/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; visual mesh filename=file:///home/mohammadnsr1/watchdog/WatchDog_V1/ros2_ws/src/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
- added link left_outer_knuckle, mass 0.05; collision mesh filename=file:///home/mohammadnsr1/watchdog/WatchDog_V1/ros2_ws/src/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; visual mesh filename=file:///home/mohammadnsr1/watchdog/WatchDog_V1/ros2_ws/src/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
- added link right_inner_finger, mass 0.05; collision mesh filename=file:///home/mohammadnsr1/watchdog/WatchDog_V1/ros2_ws/src/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; visual mesh filename=file:///home/mohammadnsr1/watchdog/WatchDog_V1/ros2_ws/src/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
- added link right_inner_knuckle, mass 0.05; collision mesh filename=file:///home/mohammadnsr1/watchdog/WatchDog_V1/ros2_ws/src/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; visual mesh filename=file:///home/mohammadnsr1/watchdog/WatchDog_V1/ros2_ws/src/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
- added link right_outer_knuckle, mass 0.05; collision mesh filename=file:///home/mohammadnsr1/watchdog/WatchDog_V1/ros2_ws/src/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; visual mesh filename=file:///home/mohammadnsr1/watchdog/WatchDog_V1/ros2_ws/src/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
- added link world
Joints:
- removed joint onrobot_rg2_base_to_body_joint
- removed joint onrobot_rg2_body_to_finger_1_origin_joint
- removed joint onrobot_rg2_body_to_finger_2_origin_joint
- removed joint onrobot_rg2_body_to_grasp_frame_joint
- removed joint onrobot_rg2_finger_1_finger_tip_to_flex_finger_joint
- removed joint onrobot_rg2_finger_1_origin_to_moment_arm_joint
- removed joint onrobot_rg2_finger_1_origin_to_truss_arm_joint
- removed joint onrobot_rg2_finger_1_truss_arm_to_finger_tip_joint
- removed joint onrobot_rg2_finger_2_finger_tip_to_flex_finger_joint
- removed joint onrobot_rg2_finger_2_origin_to_moment_arm_joint
- removed joint onrobot_rg2_finger_2_origin_to_truss_arm_joint
- removed joint onrobot_rg2_finger_2_truss_arm_to_finger_tip_joint
- added joint finger_joint: type revolute, parent base_link, child left_outer_knuckle, origin xyz=0 -0.017178 0.125797 rpy=0 0 0, axis -1 0 0, limit lower=-0.558505 upper=0.785398 effort=1000 velocity=100.0
- added joint joint0: type fixed, parent world, child base_link, origin xyz=0. 0. 0. rpy=0. 0. 1.57
- added joint left_inner_finger_joint: type revolute, parent left_outer_knuckle, child left_inner_finger, origin xyz=0 -0.039592 0.038177 rpy=0 0 0, axis 1 0 0, limit lower=-0.872665 upper=0.872665 effort=1000 velocity=100.0, mimic joint=finger_joint multiplier=1 offset=0
- added joint left_inner_knuckle_joint: type revolute, parent base_link, child left_inner_knuckle, origin xyz=0 -0.007678 0.1422970 rpy=0 0 0, axis 1 0 0, limit lower=-0.785398 upper=0.785398 effort=1000 velocity=100.0, mimic joint=finger_joint multiplier=-1 offset=0
- added joint right_inner_finger_joint: type revolute, parent right_outer_knuckle, child right_inner_finger, origin xyz=0 -0.039592 0.038177 rpy=0 0 0, axis 1 0 0, limit lower=-0.872665 upper=0.872665 effort=1000 velocity=100.0, mimic joint=finger_joint multiplier=1 offset=0
- added joint right_inner_knuckle_joint: type revolute, parent base_link, child right_inner_knuckle, origin xyz=0 0.007678 0.1422970 rpy=0 0 -3.141592653589793, axis 1 0 0, limit lower=-0.785398 upper=0.785398 effort=1000 velocity=100.0, mimic joint=finger_joint multiplier=-1 offset=0
- added joint right_outer_knuckle_joint: type revolute, parent base_link, child right_outer_knuckle, origin xyz=0 0.017178 0.125797 rpy=0 0 3.141592653589793, axis 1 0 0, limit lower=-0.785398 upper=0.785398 effort=1000 velocity=100.0, mimic joint=finger_joint multiplier=-1 offset=0

File: ros2_ws/src/robot_description/urdf/ur5e_ros.urdf (robot description, URDF)
Before this commit: robot ur5e, 22 links, 21 joints
Links:
- removed link onrobot_rg2_body_link
- removed link onrobot_rg2_finger_1_finger_tip_link
- removed link onrobot_rg2_finger_1_flex_finger_link
- removed link onrobot_rg2_finger_1_moment_arm_link
- removed link onrobot_rg2_finger_1_origin
- removed link onrobot_rg2_finger_1_truss_arm_link
- removed link onrobot_rg2_finger_2_finger_tip_link
- removed link onrobot_rg2_finger_2_flex_finger_link
- removed link onrobot_rg2_finger_2_moment_arm_link
- removed link onrobot_rg2_finger_2_origin
- removed link onrobot_rg2_finger_2_truss_arm_link
- removed link onrobot_rg2_grasp_frame
- added link onrobot_rg2_left_inner_finger, mass 0.05; collision mesh filename=package://onrobot_rg_description/meshes/rg2/collision/inner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; visual mesh filename=package://onrobot_rg_description/meshes/rg2/visual/inner_fi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
- added link onrobot_rg2_left_inner_knuckle, mass 0.05; collision mesh filename=package://onrobot_rg_description/meshes/rg2/collision/inner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; visual mesh filename=package://onrobot_rg_description/meshes/rg2/visual/inner_kn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
- added link onrobot_rg2_left_outer_knuckle, mass 0.05; collision mesh filename=package://onrobot_rg_description/meshes/rg2/collision/outer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; visual mesh filename=package://onrobot_rg_description/meshes/rg2/visual/outer_kn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
- added link onrobot_rg2_right_inner_finger, mass 0.05; collision mesh filename=package://onrobot_rg_description/meshes/rg2/collision/inner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; visual mesh filename=package://onrobot_rg_description/meshes/rg2/visual/inner_fi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
- added link onrobot_rg2_right_inner_knuckle, mass 0.05; collision mesh filename=package://onrobot_rg_description/meshes/rg2/collision/inner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; visual mesh filename=package://onrobot_rg_description/meshes/rg2/visual/inner_kn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
- added link onrobot_rg2_right_outer_knuckle, mass 0.05; collision mesh filename=package://onrobot_rg_description/meshes/rg2/collision/outer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; visual mesh filename=package://onrobot_rg_description/meshes/rg2/visual/outer_kn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
- link onrobot_rg2_base_link: mass 0.09 -> 0.7; geometry collision mesh filename=package://onrobot_rg_description/meshes/rg2/collision/base_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; visual mesh filename=package://onrobot_rg_description/meshes/rg2/visual/base_lin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
Joints:
- removed joint onrobot_rg2_base_to_body_joint
- removed joint onrobot_rg2_body_to_finger_1_origin_joint
- removed joint onrobot_rg2_body_to_finger_2_origin_joint
- removed joint onrobot_rg2_body_to_grasp_frame_joint
- removed joint onrobot_rg2_finger_1_finger_tip_to_flex_finger_joint
- removed joint onrobot_rg2_finger_1_origin_to_moment_arm_joint
- removed joint onrobot_rg2_finger_1_origin_to_truss_arm_joint
- removed joint onrobot_rg2_finger_1_truss_arm_to_finger_tip_joint
- removed joint onrobot_rg2_finger_2_finger_tip_to_flex_finger_joint
- removed joint onrobot_rg2_finger_2_origin_to_moment_arm_joint
- removed joint onrobot_rg2_finger_2_origin_to_truss_arm_joint
- removed joint onrobot_rg2_finger_2_truss_arm_to_finger_tip_joint
- added joint finger_joint: type revolute, parent onrobot_rg2_base_link, child onrobot_rg2_left_outer_knuckle, origin xyz=0 -0.017178 0.125797 rpy=0 0 0, axis -1 0 0, limit lower=-0.558505 upper=0.785398 effort=1000 velocity=100.0
- added joint left_inner_finger_joint: type revolute, parent onrobot_rg2_left_outer_knuckle, child onrobot_rg2_left_inner_finger, origin xyz=0 -0.039592 0.038177 rpy=0 0 0, axis 1 0 0, limit lower=-0.872665 upper=0.872665 effort=1000 velocity=100.0, mimic joint=finger_joint multiplier=1 offset=0
- added joint left_inner_knuckle_joint: type revolute, parent onrobot_rg2_base_link, child onrobot_rg2_left_inner_knuckle, origin xyz=0 -0.007678 0.1422970 rpy=0 0 0, axis 1 0 0, limit lower=-0.785398 upper=0.785398 effort=1000 velocity=100.0, mimic joint=finger_joint multiplier=-1 offset=0
- added joint right_inner_finger_joint: type revolute, parent onrobot_rg2_right_outer_knuckle, child onrobot_rg2_right_inner_finger, origin xyz=0 -0.039592 0.038177 rpy=0 0 0, axis 1 0 0, limit lower=-0.872665 upper=0.872665 effort=1000 velocity=100.0, mimic joint=finger_joint multiplier=1 offset=0
- added joint right_inner_knuckle_joint: type revolute, parent onrobot_rg2_base_link, child onrobot_rg2_right_inner_knuckle, origin xyz=0 0.007678 0.1422970 rpy=0 0 -3.141592653589793, axis 1 0 0, limit lower=-0.785398 upper=0.785398 effort=1000 velocity=100.0, mimic joint=finger_joint multiplier=-1 offset=0
- added joint right_outer_knuckle_joint: type revolute, parent onrobot_rg2_base_link, child onrobot_rg2_right_outer_knuckle, origin xyz=0 0.017178 0.125797 rpy=0 0 3.141592653589793, axis 1 0 0, limit lower=-0.785398 upper=0.785398 effort=1000 velocity=100.0, mimic joint=finger_joint multiplier=-1 offset=0
- joint Gripper_joint: origin xyz=0 0 0.0 rpy=0 0 0 -> xyz=0 0 0.0 rpy=0 0 -1.5707963267948966

Commit message: Update RG2 USD and URDF files for improved compatibility and structure. Add a new backup URDF file for RG2, modify existing URDF links to match final naming conventions, and update configuration USD files for consistency with recent simulation changes.

File: generated_urdf/rg2_only/rg2_only_isaac.urdf (robot description, URDF)
Before this commit: robot onrobot_rg2, 8 links, 7 joints
Links:
- removed link base_link
- removed link left_inner_finger
- removed link left_inner_knuckle
- removed link left_outer_knuckle
- removed link right_inner_finger
- removed link right_inner_knuckle
- removed link right_outer_knuckle
- added link onrobot_rg2_base_link, mass 0.7; collision mesh filename=file:///home/mohammadnsr1/watchdog/WatchDog_V1/ros2_ws/src/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; visual mesh filename=file:///home/mohammadnsr1/watchdog/WatchDog_V1/ros2_ws/src/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
- added link onrobot_rg2_left_inner_finger, mass 0.05; collision mesh filename=file:///home/mohammadnsr1/watchdog/WatchDog_V1/ros2_ws/src/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; visual mesh filename=file:///home/mohammadnsr1/watchdog/WatchDog_V1/ros2_ws/src/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
- added link onrobot_rg2_left_inner_knuckle, mass 0.05; collision mesh filename=file:///home/mohammadnsr1/watchdog/WatchDog_V1/ros2_ws/src/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; visual mesh filename=file:///home/mohammadnsr1/watchdog/WatchDog_V1/ros2_ws/src/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
- added link onrobot_rg2_left_outer_knuckle, mass 0.05; collision mesh filename=file:///home/mohammadnsr1/watchdog/WatchDog_V1/ros2_ws/src/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; visual mesh filename=file:///home/mohammadnsr1/watchdog/WatchDog_V1/ros2_ws/src/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
- added link onrobot_rg2_right_inner_finger, mass 0.05; collision mesh filename=file:///home/mohammadnsr1/watchdog/WatchDog_V1/ros2_ws/src/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; visual mesh filename=file:///home/mohammadnsr1/watchdog/WatchDog_V1/ros2_ws/src/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
- added link onrobot_rg2_right_inner_knuckle, mass 0.05; collision mesh filename=file:///home/mohammadnsr1/watchdog/WatchDog_V1/ros2_ws/src/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; visual mesh filename=file:///home/mohammadnsr1/watchdog/WatchDog_V1/ros2_ws/src/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
- added link onrobot_rg2_right_outer_knuckle, mass 0.05; collision mesh filename=file:///home/mohammadnsr1/watchdog/WatchDog_V1/ros2_ws/src/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; visual mesh filename=file:///home/mohammadnsr1/watchdog/WatchDog_V1/ros2_ws/src/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
Joints:
- joint finger_joint: child left_outer_knuckle -> onrobot_rg2_left_outer_knuckle; parent base_link -> onrobot_rg2_base_link
- joint joint0: child base_link -> onrobot_rg2_base_link
- joint left_inner_finger_joint: child left_inner_finger -> onrobot_rg2_left_inner_finger; parent left_outer_knuckle -> onrobot_rg2_left_outer_knuckle
- joint left_inner_knuckle_joint: child left_inner_knuckle -> onrobot_rg2_left_inner_knuckle; parent base_link -> onrobot_rg2_base_link
- joint right_inner_finger_joint: child right_inner_finger -> onrobot_rg2_right_inner_finger; parent right_outer_knuckle -> onrobot_rg2_right_outer_knuckle
- joint right_inner_knuckle_joint: child right_inner_knuckle -> onrobot_rg2_right_inner_knuckle; parent base_link -> onrobot_rg2_base_link
- joint right_outer_knuckle_joint: child right_outer_knuckle -> onrobot_rg2_right_outer_knuckle; parent base_link -> onrobot_rg2_base_link
