Commit message: Update UR5e URDF to correct mesh file path and modify assembly room USD file

File: config/ur5e.urdf (robot description, URDF)
Before this commit: robot ur5e, 8 links, 7 joints
Links:
- link shoulder_link: geometry collision mesh filename=file:///home/mohammadnsr1/watchdog/WatchDog_V1/assets/ur_as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; visual mesh filename=file:///home/mohammadnsr1/watchdog/WatchDog_V1/assets/ur_as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

Commit message: Update TCP joint position in URDF files for UR5e robot configuration
This commit modifies the origin position of the TCP joint in both the `ur5e.urdf` and `ur5e_ros.urdf` files, changing the z-coordinate from 0.2 to 0.15. This adjustment aims to improve the accuracy of the robot's end effector positioning.

File: config/ur5e.urdf (robot description, URDF)
Before this commit: robot ur5e, 8 links, 7 joints
Joints:
- joint wrist_3_link_to_TCP: origin xyz=0 0 0.2 rpy=0 0 0 -> xyz=0 0 0.15 rpy=0 0 0

File: ros2_ws/src/robot_description/urdf/ur5e_ros.urdf (robot description, URDF)
Before this commit: robot ur5e, 16 links, 15 joints
Joints:
- joint wrist_3_link_to_TCP: origin xyz=0 0 0.2 rpy=0 0 0 -> xyz=0 0 0.15 rpy=0 0 0
