Commit message: Add OnRobot RG2 links and joints to UR5e URDF for enhanced robotic arm functionality, including visual and collision geometries, inertial properties, and fixed joints for gripper integration.

File: ros2_ws/src/robot_description/urdf/ur5e_ros.urdf (robot description, URDF)
Before this commit: robot ur5e, 9 links, 8 joints
Links:
- added link onrobot_rg2_base_link, mass 1e-6
- added link onrobot_rg2_body_link, mass 0.65; collision mesh filename=package://onrobot_description/meshes/rg2_v1/collision/body.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; visual mesh filename=package://onrobot_description/meshes/rg2_v1/visual/body.stl
- added link onrobot_rg2_bracket_link, mass 0.09; collision mesh filename=package://onrobot_description/meshes/rg2_v1/collision/singl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; visual mesh filename=package://onrobot_description/meshes/rg2_v1/visual/single_b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
- added link onrobot_rg2_finger_1_finger_tip_link, mass 0.001; collision mesh filename=package://onrobot_description/meshes/rg2_v1/collision/finge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; visual mesh filename=package://onrobot_description/meshes/rg2_v1/visual/finger_t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
- added link onrobot_rg2_finger_1_flex_finger_link, mass 0.001; collision mesh filename=package://onrobot_description/meshes/rg2_v1/collision/flex_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; visual mesh filename=package://onrobot_description/meshes/rg2_v1/visual/flex_fin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
- added link onrobot_rg2_finger_1_moment_arm_link, mass 0.001; collision mesh filename=package://onrobot_description/meshes/rg2_v1/collision/momen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; visual mesh filename=package://onrobot_description/meshes/rg2_v1/visual/moment_a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
- added link onrobot_rg2_finger_1_origin, mass 0.001
- added link onrobot_rg2_finger_1_truss_arm_link, mass 0.001; collision mesh filename=package://onrobot_description/meshes/rg2_v1/collision/truss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; visual mesh filename=package://onrobot_description/meshes/rg2_v1/visual/truss_ar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
- added link onrobot_rg2_finger_2_finger_tip_link, mass 0.001; collision mesh filename=package://onrobot_description/meshes/rg2_v1/collision/finge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; visual mesh filename=package://onrobot_description/meshes/rg2_v1/visual/finger_t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
- added link onrobot_rg2_finger_2_flex_finger_link, mass 0.001; collision mesh filename=package://onrobot_description/meshes/rg2_v1/collision/flex_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; visual mesh filename=package://onrobot_description/meshes/rg2_v1/visual/flex_fin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
- added link onrobot_rg2_finger_2_moment_arm_link, mass 0.001; collision mesh filename=package://onrobot_description/meshes/rg2_v1/collision/momen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; visual mesh filename=package://onrobot_description/meshes/rg2_v1/visual/moment_a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
- added link onrobot_rg2_finger_2_origin, mass 0.001
- added link onrobot_rg2_finger_2_truss_arm_link, mass 0.001; collision mesh filename=package://onrobot_description/meshes/rg2_v1/collision/truss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; visual mesh filename=package://onrobot_description/meshes/rg2_v1/visual/truss_ar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
- added link onrobot_rg2_grasp_frame, mass 1e-6
Joints:
- added joint Gripper_joint: type fixed, parent wrist_3_link, child onrobot_rg2_base_link, origin xyz=0 0 0 rpy=0 0 0
- added joint onrobot_rg2_base_to_bracket_joint: type fixed, parent onrobot_rg2_base_link, child onrobot_rg2_bracket_link, origin xyz=0 0 0 rpy=0 0 0
- added joint onrobot_rg2_body_to_finger_1_origin_joint: type fixed, parent onrobot_rg2_body_link, child onrobot_rg2_finger_1_origin, origin xyz=0 0 0 rpy=0 0 0
- added joint onrobot_rg2_body_to_finger_2_origin_joint: type fixed, parent onrobot_rg2_body_link, child onrobot_rg2_finger_2_origin, origin xyz=0 0 0 rpy=0 0 3.141592653589793
- added joint onrobot_rg2_body_to_grasp_frame_joint: type fixed, parent onrobot_rg2_body_link, child onrobot_rg2_grasp_frame, origin xyz=0 0 0.14 rpy=0 0 0
- added joint onrobot_rg2_bracket_to_body_joint: type fixed, parent onrobot_rg2_bracket_link, child onrobot_rg2_body_link, origin xyz=0 0 0.05 rpy=0 0 0
- added joint onrobot_rg2_finger_1_finger_tip_to_flex_finger_joint: type fixed, parent onrobot_rg2_finger_1_finger_tip_link, child onrobot_rg2_finger_1_flex_finger_link, origin xyz=0.03059 0 0.0172 rpy=0 0 0
- added joint onrobot_rg2_finger_1_origin_to_moment_arm_joint: type fixed, parent onrobot_rg2_finger_1_origin, child onrobot_rg2_finger_1_moment_arm_link, origin xyz=-0.017 0 0.055 rpy=0 -0.772 0
- added joint onrobot_rg2_finger_1_origin_to_truss_arm_joint: type fixed, parent onrobot_rg2_finger_1_origin, child onrobot_rg2_finger_1_truss_arm_link, origin xyz=-0.0075 0 0.0715 rpy=0 -0.772 0
- added joint onrobot_rg2_finger_1_truss_arm_to_finger_tip_joint: type fixed, parent onrobot_rg2_finger_1_truss_arm_link, child onrobot_rg2_finger_1_finger_tip_link, origin xyz=-0.0256 0 0.04868 rpy=0 0.772 0
- added joint onrobot_rg2_finger_2_finger_tip_to_flex_finger_joint: type fixed, parent onrobot_rg2_finger_2_finger_tip_link, child onrobot_rg2_finger_2_flex_finger_link, origin xyz=0.03059 0 0.0172 rpy=0 0 0
- added joint onrobot_rg2_finger_2_origin_to_moment_arm_joint: type fixed, parent onrobot_rg2_finger_2_origin, child onrobot_rg2_finger_2_moment_arm_link, origin xyz=-0.017 0 0.055 rpy=0 -0.772 0
- added joint onrobot_rg2_finger_2_origin_to_truss_arm_joint: type fixed, parent onrobot_rg2_finger_2_origin, child onrobot_rg2_finger_2_truss_arm_link, origin xyz=-0.0075 0 0.0715 rpy=0 -0.772 0
- added joint onrobot_rg2_finger_2_truss_arm_to_finger_tip_joint: type fixed, parent onrobot_rg2_finger_2_truss_arm_link, child onrobot_rg2_finger_2_finger_tip_link, origin xyz=-0.0256 0 0.04868 rpy=0 0.772 0

Commit message: Update UR5e URDF and SRDF files to refine OnRobot RG2 link properties, including updated mesh paths and added collision settings for improved robot interaction.

File: ros2_ws/src/robot_description/urdf/ur5e_ros.urdf (robot description, URDF)
Before this commit: robot ur5e, 23 links, 22 joints
Links:
- removed link onrobot_rg2_bracket_link
- link onrobot_rg2_base_link: mass 1e-6 -> 0.09; geometry collision mesh filename=package://robot_description/meshes/onrobot_rg2ft/collision/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 scale=0.001 0.001 0.001; visual mesh filename=package://robot_description/meshes/onrobot_rg2ft/visual/ang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 scale=0.001 0.001 0.001

Commit message: Add fixed joint 'world_to_base_link' to UR5e URDF for base link attachment. Update move_group.launch.py to support occupancy map updates with new YAML configuration and refactor launch setup for improved parameter handling.

File: ros2_ws/src/robot_description/urdf/ur5e_ros.urdf (robot description, URDF)
Before this commit: robot ur5e, 22 links, 21 joints
Joints:
- joint world_to_base_link: origin xyz=0 0 0 rpy=0 0 0 -> xyz=0 -0.7 0 rpy=0 0 0

Commit message: Update RG2 joint limits in URDF and YAML configurations; enhance collision printing script with joint state reporting and contact pair counting. Modify RViz configuration for improved usability and adjust assembly_room.usd for compatibility with recent simulation changes.

File: ros2_ws/src/robot_description/urdf/ur5e_ros.urdf (robot description, URDF)
Before this commit: robot ur5e, 22 links, 21 joints
Joints:
- joint Gripper_joint: origin xyz=0 0 0 rpy=0 0 0 -> xyz=0 0 0.0 rpy=0 0 0
- joint onrobot_rg2_body_to_finger_2_origin_joint: origin xyz=0 0 0 rpy=0 0 3.141592653589793 -> xyz=0 0 0 rpy=0 0 -3.141592653589793
- joint onrobot_rg2_finger_1_origin_to_moment_arm_joint: limit lower=0.0 upper=1.3 effort=10.0 velocity=50.0 -> lower=0.0 upper=1.218 effort=10.0 velocity=50.0
- joint onrobot_rg2_finger_1_origin_to_truss_arm_joint: limit lower=0.0 upper=1.3 effort=10.0 velocity=50.0 -> lower=0.0 upper=1.218 effort=10.0 velocity=50.0
- joint onrobot_rg2_finger_1_truss_arm_to_finger_tip_joint: limit lower=0.0 upper=1.3 effort=10.0 velocity=50.0 -> lower=0.0 upper=1.218 effort=10.0 velocity=50.0
- joint onrobot_rg2_finger_2_origin_to_moment_arm_joint: limit lower=0.0 upper=1.3 effort=10.0 velocity=50.0 -> lower=0.0 upper=1.218 effort=10.0 velocity=50.0
- joint onrobot_rg2_finger_2_origin_to_truss_arm_joint: limit lower=0.0 upper=1.3 effort=10.0 velocity=50.0 -> lower=0.0 upper=1.218 effort=10.0 velocity=50.0
- joint onrobot_rg2_finger_2_truss_arm_to_finger_tip_joint: limit lower=0.0 upper=1.3 effort=10.0 velocity=50.0 -> lower=0.0 upper=1.218 effort=10.0 velocity=50.0

Commit message: Update assembly_room.usd, add vention.usd, and modify URDF and camera configurations
This commit includes a binary update to the assembly_room.usd file, reflecting asset changes. A new vention.usd file is added to the project. Additionally, the URDF for the UR5e robot is updated to adjust the origin of the world_to_base_link joint, and the camera settings in cameras.yaml are modified for improved positioning and orientation.

File: ros2_ws/src/robot_description/urdf/ur5e_ros.urdf (robot description, URDF)
Before this commit: robot ur5e, 16 links, 15 joints
Joints:
- joint world_to_base_link: origin xyz=0 -0.7 0 rpy=0 0 0 -> xyz=0.22686 -0.64727 0.08579 rpy=0 0 0
